File: PCB_Design/Main_Board_ONAGA/Main_Board_ONAGA.kicad_pcb (KiCad board)
At the start: 2 copper layers, 50 x 50 mm, 41 parts, among them J1 FTDI, J10 Conn, J11 Conn, J12 Conn, J2 V+-, J3 MOTOR_PINM1A, J4 MOTOR_PINM1B, J5 MOTOR_PINM1A, J6 MOTOR_PINM1B, J7 Conn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

Commit message: Diseño de PCB en proceso
Parts:
- BOOT1, EN1: footprint Button_Switch_THT:SW_PUSH_6mm_H5mm -> Button_Switch_SMD:SW_SPST_B3U-1000P
- C4, C6: moved to B.Cu
- R1, R2: moved to F.Cu
- U5, U6: footprint EESTN5-v2:SSOP-8 -> EESTN5-v2:SSOP-8_disipa
- moved EN1 37.0 mm to (148.4, 68.3), turned to 90 degrees
- moved R2 30.0 mm to (143.6, 68.6), turned to 90 degrees
- moved C3 25.9 mm to (144.9, 84.3), turned to 180 degrees
- moved U2 14.8 mm to (143.6, 78.1)
- moved J2 14.7 mm to (134.6, 107.8)
- moved C5 13.7 mm to (144.8, 72.3), turned to 0 degrees
- moved R1 10.6 mm to (126.2, 68.6), turned to -90 degrees
- moved C4 10.2 mm to (156.7, 93.9)
- moved SW3 9.98 mm to (121.2, 80.9)
- moved SW2 9.98 mm to (121.2, 88.6)
- moved R6 9.86 mm to (117.9, 86.4), turned to 180 degrees
- moved R7 9.79 mm to (117.9, 78.6), turned to 180 degrees
- moved C11 9.58 mm to (152.7, 99.7)
- moved U6 9.51 mm to (145.8, 97.7)
- moved C12 9.15 mm to (150.2, 100.7)
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Connections:
- J1 pad 3: /Rx -> /Tx
- J1 pad 4: /Tx -> /Rx
- R3 pad 1: /LED_2 -> /LED_BUILTING
- R5 pad 1: /LED_BUILTING -> /LED_2
- U1 pad 12: unconnected-(U1-IO27-Pad12) -> /M2B
- U1 pad 16: unconnected-(U1-IO13-Pad16) -> /M2A
- U1 pad 30: /BUZZER -> unconnected-(U1-IO18-Pad30)
- U1 pad 31: /M1A -> /M1B
- U1 pad 33: /M1B -> /M1A
- U1 pad 36: /M2A -> unconnected-(U1-IO22-Pad36)
- U1 pad 37: /M2B -> unconnected-(U1-IO23-Pad37)
- U6 pad 2: /M1A -> /M2A
- U6 pad 3: /M1B -> /M2B
Routing:
- net GND: track 0.00 -> 146.2 mm
- net +3V3: track 0.00 -> 68.4 mm, vias 0 -> 1
- net +5V: track 0.00 -> 52.9 mm
- net /M1A: track 0.00 -> 36.1 mm, vias 0 -> 2
- net /M1B: track 0.00 -> 30.6 mm, vias 0 -> 2
- net /PUSH_1: track 0.00 -> 21.5 mm
- net /BOOT: track 0.00 -> 21.4 mm, vias 0 -> 1
- net /LED_2: track 0.00 -> 20.8 mm, vias 0 -> 1
- net /LED_1: track 0.00 -> 19.9 mm, vias 0 -> 1
- net /M2B: track 0.00 -> 19.5 mm
- net /EN: track 0.00 -> 16.8 mm, vias 0 -> 1
- net /M2A: track 0.00 -> 16.4 mm
- net /PUSH_2: track 0.00 -> 15.4 mm
- net /Rx: track 0.00 -> 12.0 mm
- net /Tx: track 0.00 -> 11.5 mm
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- added copper zone on B.Cu, net GND
- added copper zone on F.Cu, net GND

Commit message: Chequeo de PCB
Parts:
- removed H1, H2: Mounting_Hole, EESTN5-v2:Separador_M3_5mm
- moved J5 1.20 mm to (143.0, 106.8)
- moved J6 1.20 mm to (147.6, 106.8)
- moved J3 0.99 mm to (118.1, 106.8)
- moved J4 0.99 mm to (122.6, 106.8)
- moved J1 0.88 mm to (115.2, 72.8)
Connections:
- C10 pad 1: /Vin -> VCC
- C11 pad 1: /Vin -> VCC
- C12 pad 1: /Vin -> VCC
- C9 pad 1: /Vin -> VCC
- U5 pad 5: /Vin -> VCC
- U6 pad 5: /Vin -> VCC
Routing:
- net +5V: track 52.9 -> 81.0 mm, vias 0 -> 1
- net GND: track 146.2 -> 162.1 mm
- net VCC: track 0.00 -> 14.4 mm
- net +3V3: track 68.4 -> 80.5 mm
- added copper zone on B.Cu, net /OUTM1A
- added copper zone on B.Cu, net /OUTM1B
- added copper zone on B.Cu, net /OUTM2A
- added copper zone on B.Cu, net /OUTM2B
- added copper zone on B.Cu, net VCC
