File: PCB_Design/Main_Board_ONAGA/Main_Board_ONAGA.kicad_sch (KiCad schematic)
At the start: 41 parts, among them J1 FTDI, J10 Conn, J11 Conn, J12 Conn, J2 V+-, J3 MOTOR_PINM1A, J4 MOTOR_PINM1B, J5 MOTOR_PINM1A, J6 MOTOR_PINM1B, J7 Conn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

Commit message: Diseño de PCB en proceso
Parts:
- BOOT1, EN1: footprint Button_Switch_THT:SW_PUSH_6mm_H5mm -> Button_Switch_SMD:SW_SPST_B3U-1000P
- U5, U6: footprint EESTN5-v2:SSOP-8 -> EESTN5-v2:SSOP-8_disipa
Connections:
- net LED_2: now also R5.1; no longer R3.1
- net LED_BUILTING: now also R3.1; no longer R5.1
- net M1A: now also U1.33 (IO21); no longer U1.31 (IO19), U6.2 (IN2)
- net M1B: now also U1.31 (IO19); no longer U1.33 (IO21), U6.3 (IN1)
- net M2A: now also U1.16 (IO13), U6.2 (IN2); no longer U1.36 (IO22)
- net M2B: now also U1.12 (IO27), U6.3 (IN1); no longer U1.37 (IO23)
- net Rx: now also J1.4 (Pin_4); no longer J1.3 (Pin_3)
- net Tx: now also J1.3 (Pin_3); no longer J1.4 (Pin_4)
- net BUZZER: no longer names the net of U1.30 (IO18)
Other:
- moved on the sheet: D1, D3, R3, R5
Changed lines of the file:
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@@
     (stroke (width 0) (type default))
   )
-  (wire (pts (xy 136.779 148.2852) (xy 136.779 152.6032))
-    (stroke (width 0) (type default))
-  )
   (wire (pts (xy 245.5418 43.9928) (xy 245.5418 45.2628))
     (stroke (width 0) (type default))
@@
     (stroke (width 0) (type default))
   )
-  (wire (pts (xy 142.8242 82.5246) (xy 146.1262 82.5246))
+  (wire (pts (xy 142.8242 90.1446) (xy 146.1262 90.1446))
     (stroke (width 0) (type default))
   )
@@
     (stroke (width 0) (type default))
   )
-  (wire (pts (xy 142.8242 79.9846) (xy 146.2532 79.9846))
+  (wire (pts (xy 142.8242 59.6646) (xy 146.2532 59.6646))
     (stroke (width 0) (type default))
   )
@@
     (stroke (width 0) (type default))
   )
-  (wire (pts (xy 142.8242 72.3646) (xy 146.1262 72.3646))
-    (stroke (width 0) (type default))
-  )
   (wire (pts (xy 71.0184 56.642) (xy 71.0184 57.658))
     (stroke (width 0) (type default))
@@
     (stroke (width 0) (type default))
   )
+  (wire (pts (xy 136.779 148.2852) (xy 136.779 152.6032))
+    (stroke (width 0) (type default))
+  )
   (wire (pts (xy 60.8076 92.5322) (xy 60.8076 89.3572))
     (stroke (width 0) (type default))
@@
     (effects (font (size 1.524 1.524)) (justify left bottom))
   )
-  (label "Tx" (at 27.3558 109.2708 0) (fields_autoplaced)
+  (label "Tx" (at 27.3558 106.7308 0) (fields_autoplaced)
     (effects (font (size 1.27 1.27)) (justify left bottom))
   )
@@
     (effects (font (size 1.524 1.524)) (justify left bottom))
   )
-  (label "M1A" (at 199.9742 83.3374 180) (fields_autoplaced)
+  (label "M2A" (at 199.9742 83.3374 180) (fields_autoplaced)
     (effects (font (size 1.524 1.524)) (justify right bottom))
   )
@@
     (effects (font (size 1.524 1.524)) (justify left bottom))
   )
-  (label "BUZZER" (at 146.1262 72.3646 0) (fields_autoplaced)
-    (effects (font (size 1.524 1.524)) (justify left bottom))
-  )
   (label "INP_2" (at 145.923 100.3046 0) (fields_autoplaced)
     (effects (font (size 1.524 1.524)) (justify left bottom))
@@
     (effects (font (size 1.524 1.524)) (justify left bottom))
   )
-  (label "Rx" (at 27.3558 106.7308 0) (fields_autoplaced)
+  (label "Rx" (at 27.3558 109.2708 0) (fields_autoplaced)
     (effects (font (size 1.27 1.27)) (justify left bottom))
   )
@@
     (effects (font (size 1.524 1.524)) (justify left bottom))
   )
-  (label "M1B" (at 146.1262 77.4446 0) (fields_autoplaced)
+  (label "M1B" (at 146.1262 74.9046 0) (fields_autoplaced)
     (effects (font (size 1.524 1.524)) (justify left bottom))
   )
@@
     (effects (font (size 1.524 1.524)) (justify left bottom))
   )
-  (label "M1A" (at 146.1262 74.9046 0) (fields_autoplaced)
+  (label "M1A" (at 146.1262 77.4446 0) (fields_autoplaced)
     (effects (font (size 1.524 1.524)) (justify left bottom))
   )
@@
     (effects (font (size 1.524 1.524)) (justify left bottom))
   )
-  (label "M2B" (at 146.1262 82.5246 0) (fields_autoplaced)
+  (label "M2B" (at 146.1262 90.1446 0) (fields_autoplaced)
     (effects (font (size 1.524 1.524)) (justify left bottom))
   )
@@
     (effects (font (size 1.524 1.524)) (justify left bottom))
   )
-  (label "M1B" (at 199.9742 85.8774 180) (fields_autoplaced)
+  (label "M2B" (at 199.9742 85.8774 180) (fields_autoplaced)
     (effects (font (size 1.524 1.524)) (justify right bottom))
   )
-  (label "M2A" (at 146.2532 79.9846 0) (fields_autoplaced)
+  (label "M2A" (at 146.2532 59.6646 0) (fields_autoplaced)
     (effects (font (size 1.524 1.524)) (justify left bottom))
   )
@@
     )
   )
-  (symbol (lib_id "Device:LED") (at 136.779 166.5732 90) (unit 1)
+  (symbol (lib_id "Device:LED") (at 116.4082 166.5732 90) (unit 1)
     (in_bom yes) (on_board yes) (dnp no)
-    (property "Reference" "D3" (at 140.843 164.7952 90)
+    (property "Reference" "D3" (at 120.4722 164.7952 90)
       (effects (font (size 1.27 1.27)))
     )
-    (property "Value" "LED" (at 140.843 167.3352 90)
+    (property "Value" "LED" (at 120.4722 167.3352 90)
       (effects (font (size 1.27 1.27)))
     )
-    (property "Footprint" "EESTN5-v2:Led_0805" (at 136.779 166.5732 0)
+    (property "Footprint" "EESTN5-v2:Led_0805" (at 116.4082 166.5732 0)
       (effects (font (size 1.27 1.27)) hide)
     )
-    (property "Datasheet" "~" (at 136.779 166.5732 0)
+    (property "Datasheet" "~" (at 116.4082 166.5732 0)
       (effects (font (size 1.27 1.27)) hide)
     )
@@
       (effects (font (size 1.524 1.524)))
     )
-    (property "Footprint" "EESTN5-v2:SSOP-8" (at 221.4118 46.5328 0)
+    (property "Footprint" "EESTN5-v2:SSOP-8_disipa" (at 221.4118 46.5328 0)
       (effects (font (size 1.524 1.524)) hide)
     )
@@
     )
   )
-  (symbol (lib_id "Device:LED") (at 116.4082 166.5732 90) (unit 1)
+  (symbol (lib_id "Device:LED") (at 136.779 166.5732 90) (unit 1)
     (in_bom yes) (on_board yes) (dnp no)
-    (property "Reference" "D1" (at 120.4722 164.7952 90)
+    (property "Reference" "D1" (at 140.843 164.7952 90)
       (effects (font (size 1.27 1.27)))
     )
-    (property "Value" "LED" (at 120.4722 167.3352 90)
+    (property "Value" "LED" (at 140.843 167.3352 90)
       (effects (font (size 1.27 1.27)))
     )
-    (property "Footprint" "EESTN5-v2:Led_0805" (at 116.4082 166.5732 0)
+    (property "Footprint" "EESTN5-v2:Led_0805" (at 136.779 166.5732 0)
       (effects (font (size 1.27 1.27)) hide)
     )
-    (property "Datasheet" "~" (at 116.4082 166.5732 0)
+    (property "Datasheet" "~" (at 136.779 166.5732 0)
       (effects (font (size 1.27 1.27)) hide)
     )
@@
       (effects (font (size 1.27 1.27)) hide)
     )
-    (property "Footprint" "Button_Switch_THT:SW_PUSH_6mm_H5mm" (at 36.322 112.8268 0)
+    (property "Footprint" "Button_Switch_SMD:SW_SPST_B3U-1000P" (at 36.322 112.8268 0)
       (effects (font (size 1.27 1.27)) hide)
     )
@@
     )
   )
-  (symbol (lib_id "Device:R") (at 116.4082 156.4132 0) (unit 1)
+  (symbol (lib_id "Device:R") (at 136.779 156.4132 0) (unit 1)
     (in_bom yes) (on_board yes) (dnp no)
-    (property "Reference" "R3" (at 117.6782 155.1432 0)
+    (property "Reference" "R3" (at 138.049 155.1432 0)
       (effects (font (size 1.27 1.27)) (justify left))
     )
-    (property "Value" "220" (at 117.6782 157.6832 0)
+    (property "Value" "220" (at 138.049 157.6832 0)
       (effects (font (size 1.27 1.27)) (justify left))
     )
-    (property "Footprint" "EESTN5-v2:R_1206" (at 114.6302 156.4132 90)
+    (property "Footprint" "EESTN5-v2:R_1206" (at 135.001 156.4132 90)
       (effects (font (size 1.27 1.27)) hide)
     )
-    (property "Datasheet" "~" (at 116.4082 156.4132 0)
+    (property "Datasheet" "~" (at 136.779 156.4132 0)
       (effects (font (size 1.27 1.27)) hide)
     )
@@
       (effects (font (size 1.524 1.524)))
     )
-    (property "Footprint" "EESTN5-v2:SSOP-8" (at 222.1992 90.9574 0)
+    (property "Footprint" "EESTN5-v2:SSOP-8_disipa" (at 222.1992 90.9574 0)
       (effects (font (size 1.524 1.524)) hide)
     )
@@
       (effects (font (size 1.27 1.27)) hide)
     )
-    (property "Footprint" "Button_Switch_THT:SW_PUSH_6mm_H5mm" (at 55.7276 112.8522 0)
+    (property "Footprint" "Button_Switch_SMD:SW_SPST_B3U-1000P" (at 55.7276 112.8522 0)
       (effects (font (size 1.27 1.27)) hide)
     )
@@
     )
   )
-  (symbol (lib_id "Device:R") (at 136.779 156.4132 0) (unit 1)
+  (symbol (lib_id "Device:R") (at 116.4082 156.4132 0) (unit 1)
     (in_bom yes) (on_board yes) (dnp no)
-    (property "Reference" "R5" (at 138.049 155.1432 0)
+    (property "Reference" "R5" (at 117.6782 155.1432 0)
       (effects (font (size 1.27 1.27)) (justify left))
     )
-    (property "Value" "220" (at 138.049 157.6832 0)
+    (property "Value" "220" (at 117.6782 157.6832 0)
       (effects (font (size 1.27 1.27)) (justify left))
     )
-    (property "Footprint" "EESTN5-v2:R_1206" (at 135.001 156.4132 90)
+    (property "Footprint" "EESTN5-v2:R_1206" (at 114.6302 156.4132 90)
       (effects (font (size 1.27 1.27)) hide)
     )
-    (property "Datasheet" "~" (at 136.779 156.4132 0)
+    (property "Datasheet" "~" (at 116.4082 156.4132 0)
       (effects (font (size 1.27 1.27)) hide)
     )

Commit message: Chequeo de PCB
Connections:
- net Vin is gone; now on net VCC: C10.1, C11.1, C12.1, C9.1, U5.5 (VM), U6.5 (VM)
Changed lines of the file:
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@@
     (stroke (width 0) (type default))
   )
+  (wire (pts (xy 248.7168 32.8168) (xy 248.7168 43.9928))
+    (stroke (width 0) (type default))
+  )
   (wire (pts (xy 219.4306 153.416) (xy 219.4306 154.686))
     (stroke (width 0) (type default))
@@
     (stroke (width 0) (type default))
   )
+  (wire (pts (xy 249.5042 77.2414) (xy 249.5042 88.4174))
+    (stroke (width 0) (type default))
+  )
   (wire (pts (xy 218.7702 131.8006) (xy 218.7702 133.0706))
     (stroke (width 0) (type default))
@@
     (effects (font (size 1.524 1.524)) (justify right bottom))
   )
-  (label "Vin" (at 248.7168 43.9928 0) (fields_autoplaced)
-    (effects (font (size 1.524 1.524)) (justify left bottom))
-  )
   (label "Rx" (at 150.3172 44.4246 0) (fields_autoplaced)
     (effects (font (size 1.27 1.27)) (justify left bottom))
   )
-  (label "Vin" (at 249.5042 88.4174 0) (fields_autoplaced)
-    (effects (font (size 1.524 1.524)) (justify left bottom))
-  )
   (label "INP_6" (at 145.8976 87.6046 0) (fields_autoplaced)
     (effects (font (size 1.524 1.524)) (justify left bottom))
@@
     )
   )
+  (symbol (lib_id "power:VCC") (at 249.5042 77.2414 0) (unit 1)
+    (in_bom yes) (on_board yes) (dnp no)
+    (property "Reference" "#PWR046" (at 249.5042 81.0514 0)
+      (effects (font (size 1.27 1.27)) hide)
+    )
+    (property "Value" "VCC" (at 249.5042 73.4314 0)
+      (effects (font (size 1.27 1.27)))
+    )
+    (property "Footprint" "" (at 249.5042 77.2414 0)
+      (effects (font (size 1.27 1.27)) hide)
+    )
+    (property "Datasheet" "" (at 249.5042 77.2414 0)
+      (effects (font (size 1.27 1.27)) hide)
+    )
+    (pin "1")
+    (instances
+      (project "Main_Board_ONAGA"
+        (path "/0e2ee51b-8ca6-4bc3-bf29-93c6145de010"
+          (reference "#PWR046") (unit 1)
+        )
+      )
+      (project "Main_Board_COYOTE"
+        (path "/8dc25483-921d-4069-82df-8c37827f2e52"
+          (reference "#PWR01") (unit 1)
+        )
+      )
+      (project "Main board - Junior"
+        (path "/e63e39d7-6ac0-4ffd-8aa3-1841a4541b55"
+          (reference "#PWR03") (unit 1)
+        )
+      )
+    )
+  )
   (symbol (lib_id "RF_Module:ESP32-WROOM-32") (at 127.5842 72.3646 0) (unit 1)
     (in_bom yes) (on_board yes) (dnp no) (fields_autoplaced)
@@
         )
       )
+    )
+  )
+  (symbol (lib_id "power:VCC") (at 248.7168 32.8168 0) (unit 1)
+    (in_bom yes) (on_board yes) (dnp no)
+    (property "Reference" "#PWR047" (at 248.7168 36.6268 0)
+      (effects (font (size 1.27 1.27)) hide)
+    )
+    (property "Value" "VCC" (at 248.7168 29.0068 0)
+      (effects (font (size 1.27 1.27)))
+    )
+    (property "Footprint" "" (at 248.7168 32.8168 0)
+      (effects (font (size 1.27 1.27)) hide)
+    )
+    (property "Datasheet" "" (at 248.7168 32.8168 0)
+      (effects (font (size 1.27 1.27)) hide)
+    )
+    (pin "1")
+    (instances
+      (project "Main_Board_ONAGA"
+        (path "/0e2ee51b-8ca6-4bc3-bf29-93c6145de010"
+          (reference "#PWR047") (unit 1)
+        )
+      )
+      (project "Main_Board_COYOTE"
+        (path "/8dc25483-921d-4069-82df-8c37827f2e52"
+          (reference "#PWR01") (unit 1)
+        )
+      )
+      (project "Main board - Junior"
+        (path "/e63e39d7-6ac0-4ffd-8aa3-1841a4541b55"
+          (reference "#PWR03") (unit 1)
+        )
+      )
